File: ui_board_1u.kicad_pcb (KiCad board)
At the start: 2 copper layers, 156 x 38 mm, 121 parts, among them J1 X9555WV-2x06-6TV01, J5 BM07B-SRSS-TB, SW1 B3FS-1052, SW2 291V1022F832AB, SW3 PEC164220F-S0024, SW4 MS-22C01-G010, U1 AFC01-S30FCA-00, U2 SPX3819M5-L, U3 TPS61040DBV, U4 MCP23S17_ML

Commit message: PCB: sync with schematic. Upgrade to kicad 10
Parts:
- C11, C12, C13, C14: value 10n -> 100n
- R12, R17: value 150R -> 1k8
- R13, R18: value 560R -> 3k6
- R14, R19: value 22R -> 910R
